Commit message: 模型替换

File: src/humanoid_control/humanoid_legged_description/urdf/humanoid_legged_control_.urdf (robot description, URDF)
Before this commit: robot humanoid-legged-description, 32 links, 31 joints
Links:
- removed link arm_l1_link
- removed link arm_l2_link
- removed link arm_l3_link
- removed link arm_l4_link
- removed link arm_l5_link
- removed link arm_l6_link
- removed link arm_r1_link
- removed link arm_r2_link
- removed link arm_r3_link
- removed link arm_r4_link
- removed link arm_r5_link
- removed link arm_r6_link
- removed link head_yaw_link
- removed link l_foot_heel
- removed link l_foot_toe
- removed link leg_l1_link
- removed link leg_l2_link
- removed link leg_l3_link
- removed link leg_l4_link
- removed link leg_l5_link
- removed link leg_l6_link
- removed link leg_r1_link
- removed link leg_r2_link
- removed link leg_r3_link
- removed link leg_r4_link
- removed link leg_r5_link
- removed link leg_r6_link
- removed link r_foot_heel
- removed link r_foot_toe
- removed link waist_yaw_link
- added link Ankle_L_Pitch_Link, mass 0.088; visual mesh filename=package://humanoid_legged_description/meshes/Ankle_L_Pitch_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
- added link Ankle_L_Roll_Link, mass 0.758; collision box size=0.25 0.1 0.025; visual mesh filename=package://humanoid_legged_description/meshes/Ankle_L_Roll_L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
- added link Ankle_R_Pitch_Link, mass 0.088; visual mesh filename=package://humanoid_legged_description/meshes/Ankle_R_Pitch_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
- added link Ankle_R_Roll_Link, mass 0.758; collision box size=0.25 0.1 0.025; visual mesh filename=package://humanoid_legged_description/meshes/Ankle_R_Roll_L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
- added link Hip_L_Pitch_Link, mass 6.22; collision box size=0.13 0.07 0.25; collision cylinder length=0.12 radius=0.08
- added link Hip_L_Roll_Link, mass 2.28; collision cylinder length=0.035 radius=0.07; collision cylinder length=0.06 radius=0.05
- added link Hip_L_Yaw_Link, mass 3.738; collision cylinder length=0.13 radius=0.07; visual mesh filename=package://humanoid_legged_description/meshes/Hip_L_Yaw_Link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
- added link Hip_R_Pitch_Link, mass 6.22; collision box size=0.13 0.07 0.25; collision cylinder length=0.12 radius=0.08
- added link Hip_R_Roll_Link, mass 2.28; collision cylinder length=0.035 radius=0.07; collision cylinder length=0.06 radius=0.05
- added link Hip_R_Yaw_Link, mass 4.801; collision cylinder length=0.13 radius=0.07; visual mesh filename=package://humanoid_legged_description/meshes/Hip_R_Yaw_Link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
- added link Knee_L_Pitch_Link, mass 3.32; collision box size=0.1 0.08 0.3; visual mesh filename=package://humanoid_legged_description/meshes/Knee_L_Pitch_L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
- added link Knee_R_Pitch_Link, mass 3.32; collision box size=0.1 0.08 0.3; visual mesh filename=package://humanoid_legged_description/meshes/Knee_R_Pitch_L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
- link base_link: mass 11.000 -> 28; geometry collision box size=0.20 0.33 0.35; collision cylinder length=0.07 radius=0.05
Joints:
- removed joint arm_l1_joint
- removed joint arm_l2_joint
- removed joint arm_l3_joint
- removed joint arm_l4_joint
- removed joint arm_l5_joint
- removed joint arm_l6_joint
- removed joint arm_r1_joint
- removed joint arm_r2_joint
- removed joint arm_r3_joint
- removed joint arm_r4_joint
- removed joint arm_r5_joint
- removed joint arm_r6_joint
- removed joint head_yaw_joint
- removed joint l_foot_heel_joint
- removed joint l_foot_toe_joint
- removed joint leg_l1_joint
- removed joint leg_l2_joint
- removed joint leg_l3_joint
- removed joint leg_l4_joint
- removed joint leg_l5_joint
- removed joint leg_l6_joint
- removed joint leg_r1_joint
- removed joint leg_r2_joint
- removed joint leg_r3_joint
- removed joint leg_r4_joint
- removed joint leg_r5_joint
- removed joint leg_r6_joint
- removed joint r_foot_heel_joint
- removed joint r_foot_toe_joint
- removed joint waist_yaw_joint
- added joint Ankle_L_Pitch_Joint: type revolute, parent Knee_L_Pitch_Link, child Ankle_L_Pitch_Link, origin xyz=0 0 -0.4 rpy=0 0 0, axis 0 1 0, limit lower=-0.78 upper=0.57 effort=200 velocity=5
- added joint Ankle_L_Roll_Joint: type revolute, parent Ankle_L_Pitch_Link, child Ankle_L_Roll_Link, origin xyz=0 0 0 rpy=0 0 0, axis 1 0 0, limit lower=-0.35 upper=0.35 effort=200 velocity=5
- added joint Ankle_R_Pitch_Joint: type revolute, parent Knee_R_Pitch_Link, child Ankle_R_Pitch_Link, origin xyz=0 0 -0.4 rpy=0 0 0, axis 0 1 0, limit lower=-0.78 upper=0.57 effort=200 velocity=5
- added joint Ankle_R_Roll_Joint: type revolute, parent Ankle_R_Pitch_Link, child Ankle_R_Roll_Link, origin xyz=0 0 0 rpy=0 0 0, axis 1 0 0, limit lower=-0.35 upper=0.35 effort=200 velocity=5
- added joint Hip_L_Pitch_Joint: type revolute, parent Hip_L_Yaw_Link, child Hip_L_Pitch_Link, origin xyz=0 0 -0.10595 rpy=0 0 0, axis 0 1 0, limit lower=-0.78 upper=0.78 effort=200 velocity=5
- added joint Hip_L_Roll_Joint: type revolute, parent base_link, child Hip_L_Roll_Link, origin xyz=-0.042 0.1275 -0.097 rpy=0 0 0, axis 1 0 0, limit lower=-0.227 upper=0.523 effort=200 velocity=5
- added joint Hip_L_Yaw_Joint: type revolute, parent Hip_L_Roll_Link, child Hip_L_Yaw_Link, origin xyz=0.087 0 -0.0135 rpy=0 0 0, axis 0 0 1, limit lower=-0.5 upper=0.65 effort=200 velocity=5
- added joint Hip_R_Pitch_Joint: type revolute, parent Hip_R_Yaw_Link, child Hip_R_Pitch_Link, origin xyz=0 0 -0.10595 rpy=0 0 0, axis 0 1 0, limit lower=-0.78 upper=0.78 effort=200 velocity=5
- added joint Hip_R_Roll_Joint: type revolute, parent base_link, child Hip_R_Roll_Link, origin xyz=-0.042 -0.1275 -0.097 rpy=0 0 0, axis 1 0 0, limit lower=-0.52 upper=0.23 effort=200 velocity=5
- added joint Hip_R_Yaw_Joint: type revolute, parent Hip_R_Roll_Link, child Hip_R_Yaw_Link, origin xyz=0.087 0 -0.0135 rpy=0 0 0, axis 0 0 1, limit lower=-0.65 upper=0.5 effort=200 velocity=5
- added joint Knee_L_Pitch_Joint: type revolute, parent Hip_L_Pitch_Link, child Knee_L_Pitch_Link, origin xyz=0 0 -0.34 rpy=0 0 0, axis 0 1 0, limit lower=0 upper=1.2 effort=200 velocity=5
- added joint Knee_R_Pitch_Joint: type revolute, parent Hip_R_Pitch_Link, child Knee_R_Pitch_Link, origin xyz=0 0 -0.34 rpy=0 0 0, axis 0 1 0, limit lower=0 upper=1.2 effort=200 velocity=5
- joint dummy_to_base_link: origin xyz=0 0 0.4005 rpy=0 0 0 -> xyz=0 0.133 0.03605 rpy=0 0 0

File: src/humanoid_control/humanoid_legged_description/urdf/humanoid_legged_origin.urdf (robot description, URDF)
Before this commit: robot humanoid_legged_description, 32 links, 31 joints
Links:
- removed link arm_l1_link
- removed link arm_l2_link
- removed link arm_l3_link
- removed link arm_l4_link
- removed link arm_l5_link
- removed link arm_l6_link
- removed link arm_r1_link
- removed link arm_r2_link
- removed link arm_r3_link
- removed link arm_r4_link
- removed link arm_r5_link
- removed link arm_r6_link
- removed link head_yaw_link
- removed link l_foot_heel
- removed link l_foot_toe
- removed link leg_l1_link
- removed link leg_l2_link
- removed link leg_l3_link
- removed link leg_l4_link
- removed link leg_l5_link
- removed link leg_l6_link
- removed link leg_r1_link
- removed link leg_r2_link
- removed link leg_r3_link
- removed link leg_r4_link
- removed link leg_r5_link
- removed link leg_r6_link
- removed link r_foot_heel
- removed link r_foot_toe
- removed link waist_yaw_link
- added link Ankle_L_Pitch_Link, mass 0.088; visual mesh filename=package://humanoid_legged_description/meshes/Ankle_L_Pitch_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
- added link Ankle_L_Roll_Link, mass 0.758; collision box size=0.25 0.1 0.025; visual mesh filename=package://humanoid_legged_description/meshes/Ankle_L_Roll_L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
- added link Ankle_R_Pitch_Link, mass 0.088; visual mesh filename=package://humanoid_legged_description/meshes/Ankle_R_Pitch_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
- added link Ankle_R_Roll_Link, mass 0.758; collision box size=0.25 0.1 0.025; visual mesh filename=package://humanoid_legged_description/meshes/Ankle_R_Roll_L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
- added link Hip_L_Pitch_Link, mass 6.22; collision box size=0.13 0.07 0.25; collision cylinder length=0.12 radius=0.08
- added link Hip_L_Roll_Link, mass 2.28; collision cylinder length=0.035 radius=0.07; collision cylinder length=0.06 radius=0.05
- added link Hip_L_Yaw_Link, mass 3.738; collision cylinder length=0.13 radius=0.07; visual mesh filename=package://humanoid_legged_description/meshes/Hip_L_Yaw_Link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
- added link Hip_R_Pitch_Link, mass 6.22; collision box size=0.13 0.07 0.25; collision cylinder length=0.12 radius=0.08
- added link Hip_R_Roll_Link, mass 2.28; collision cylinder length=0.035 radius=0.07; collision cylinder length=0.06 radius=0.05
- added link Hip_R_Yaw_Link, mass 4.801; collision cylinder length=0.13 radius=0.07; visual mesh filename=package://humanoid_legged_description/meshes/Hip_R_Yaw_Link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
- added link Knee_L_Pitch_Link, mass 3.32; collision box size=0.1 0.08 0.3; visual mesh filename=package://humanoid_legged_description/meshes/Knee_L_Pitch_L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
- added link Knee_R_Pitch_Link, mass 3.32; collision box size=0.1 0.08 0.3; visual mesh filename=package://humanoid_legged_description/meshes/Knee_R_Pitch_L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
- link base_link: mass 11.000 -> 28; geometry collision box size=0.20 0.33 0.35; collision cylinder length=0.07 radius=0.05
Joints:
- removed joint arm_l1_joint
- removed joint arm_l2_joint
- removed joint arm_l3_joint
- removed joint arm_l4_joint
- removed joint arm_l5_joint
- removed joint arm_l6_joint
- removed joint arm_r1_joint
- removed joint arm_r2_joint
- removed joint arm_r3_joint
- removed joint arm_r4_joint
- removed joint arm_r5_joint
- removed joint arm_r6_joint
- removed joint head_yaw_joint
- removed joint l_foot_heel_joint
- removed joint l_foot_toe_joint
- removed joint leg_l1_joint
- removed joint leg_l2_joint
- removed joint leg_l3_joint
- removed joint leg_l4_joint
- removed joint leg_l5_joint
- removed joint leg_l6_joint
- removed joint leg_r1_joint
- removed joint leg_r2_joint
- removed joint leg_r3_joint
- removed joint leg_r4_joint
- removed joint leg_r5_joint
- removed joint leg_r6_joint
- removed joint r_foot_heel_joint
- removed joint r_foot_toe_joint
- removed joint waist_yaw_joint
- added joint Ankle_L_Pitch_Joint: type revolute, parent Knee_L_Pitch_Link, child Ankle_L_Pitch_Link, origin xyz=0 0 -0.4 rpy=0 0 0, axis 0 1 0, limit lower=-0.78 upper=0.57 effort=200 velocity=5
- added joint Ankle_L_Roll_Joint: type revolute, parent Ankle_L_Pitch_Link, child Ankle_L_Roll_Link, origin xyz=0 0 0 rpy=0 0 0, axis 1 0 0, limit lower=-0.35 upper=0.35 effort=200 velocity=5
- added joint Ankle_R_Pitch_Joint: type revolute, parent Knee_R_Pitch_Link, child Ankle_R_Pitch_Link, origin xyz=0 0 -0.4 rpy=0 0 0, axis 0 1 0, limit lower=-0.78 upper=0.57 effort=200 velocity=5
- added joint Ankle_R_Roll_Joint: type revolute, parent Ankle_R_Pitch_Link, child Ankle_R_Roll_Link, origin xyz=0 0 0 rpy=0 0 0, axis 1 0 0, limit lower=-0.35 upper=0.35 effort=200 velocity=5
- added joint Hip_L_Pitch_Joint: type revolute, parent Hip_L_Yaw_Link, child Hip_L_Pitch_Link, origin xyz=0 0 -0.10595 rpy=0 0 0, axis 0 1 0, limit lower=-0.78 upper=0.78 effort=200 velocity=5
- added joint Hip_L_Roll_Joint: type revolute, parent base_link, child Hip_L_Roll_Link, origin xyz=-0.042 0.1275 -0.097 rpy=0 0 0, axis 1 0 0, limit lower=-0.227 upper=0.523 effort=200 velocity=5
- added joint Hip_L_Yaw_Joint: type revolute, parent Hip_L_Roll_Link, child Hip_L_Yaw_Link, origin xyz=0.087 0 -0.0135 rpy=0 0 0, axis 0 0 1, limit lower=-0.5 upper=0.65 effort=200 velocity=5
- added joint Hip_R_Pitch_Joint: type revolute, parent Hip_R_Yaw_Link, child Hip_R_Pitch_Link, origin xyz=0 0 -0.10595 rpy=0 0 0, axis 0 1 0, limit lower=-0.78 upper=0.78 effort=200 velocity=5
- added joint Hip_R_Roll_Joint: type revolute, parent base_link, child Hip_R_Roll_Link, origin xyz=-0.042 -0.1275 -0.097 rpy=0 0 0, axis 1 0 0, limit lower=-0.52 upper=0.23 effort=200 velocity=5
- added joint Hip_R_Yaw_Joint: type revolute, parent Hip_R_Roll_Link, child Hip_R_Yaw_Link, origin xyz=0.087 0 -0.0135 rpy=0 0 0, axis 0 0 1, limit lower=-0.65 upper=0.5 effort=200 velocity=5
- added joint Knee_L_Pitch_Joint: type revolute, parent Hip_L_Pitch_Link, child Knee_L_Pitch_Link, origin xyz=0 0 -0.34 rpy=0 0 0, axis 0 1 0, limit lower=0 upper=1.2 effort=200 velocity=5
- added joint Knee_R_Pitch_Joint: type revolute, parent Hip_R_Pitch_Link, child Knee_R_Pitch_Link, origin xyz=0 0 -0.34 rpy=0 0 0, axis 0 1 0, limit lower=0 upper=1.2 effort=200 velocity=5
- joint dummy_to_base_link: origin xyz=0 0 0.4005 rpy=0 0 0 -> xyz=0 0.133 0.03605 rpy=0 0 0

Commit message: 基本跑通，正在改

File: src/humanoid_control/humanoid_legged_description/urdf/humanoid_legged_control_.urdf (robot description, URDF)
Before this commit: robot humanoid_legged_description, 14 links, 13 joints
Links:
- added link l_foot_heel
- added link l_foot_toe
- added link r_foot_heel
- added link r_foot_toe
Joints:
- added joint l_foot_heel_joint: type fixed, parent Ankle_L_Roll_Link, child l_foot_heel, origin xyz=-0.08326  0 -0.068 rpy=0 0 0
- added joint l_foot_toe_joint: type fixed, parent Ankle_L_Roll_Link, child l_foot_toe, origin xyz=0.15484 0 -0.068 rpy=0 0 0
- added joint r_foot_heel_joint: type fixed, parent Ankle_R_Roll_Link, child r_foot_heel, origin xyz=-0.08326  0 -0.068 rpy=0 0 0
- added joint r_foot_toe_joint: type fixed, parent Ankle_R_Roll_Link, child r_foot_toe, origin xyz=0.15484 0 -0.068 rpy=0 0 0

Commit message: 修改脚底接触点，现存dummyLink问题

File: src/humanoid_control/humanoid_legged_description/urdf/humanoid_legged_control_.urdf (robot description, URDF)
Before this commit: robot humanoid_legged_description, 18 links, 17 joints
Joints:
- joint dummy_to_base_link: origin xyz=0 0.133 0.03605 rpy=0 0 0 -> xyz=-0.3605 0 -0.133 rpy=0 0 0
- joint l_foot_heel_joint: origin xyz=-0.08326  0 -0.068 rpy=0 0 0 -> xyz=-0.08326  0 -0.0725 rpy=0 0 0
- joint l_foot_toe_joint: origin xyz=0.15484 0 -0.068 rpy=0 0 0 -> xyz=0.15484 0 -0.0725 rpy=0 0 0
- joint r_foot_heel_joint: origin xyz=-0.08326  0 -0.068 rpy=0 0 0 -> xyz=-0.08326  0 -0.0725 rpy=0 0 0
- joint r_foot_toe_joint: origin xyz=0.15484 0 -0.068 rpy=0 0 0 -> xyz=0.15484 0 -0.0725 rpy=0 0 0

File: src/humanoid_control/humanoid_legged_description/urdf/humanoid_legged_origin.urdf (robot description, URDF)
Before this commit: robot humanoid_legged_description, 14 links, 13 joints
Links:
- added link l_foot_heel
- added link l_foot_toe
- added link r_foot_heel
- added link r_foot_toe
Joints:
- added joint l_foot_heel_joint: type fixed, parent Ankle_L_Roll_Link, child l_foot_heel, origin xyz=-0.08326  0 -0.0725 rpy=0 0 0
- added joint l_foot_toe_joint: type fixed, parent Ankle_L_Roll_Link, child l_foot_toe, origin xyz=0.15484 0 -0.0725 rpy=0 0 0
- added joint r_foot_heel_joint: type fixed, parent Ankle_R_Roll_Link, child r_foot_heel, origin xyz=-0.08326  0 -0.0725 rpy=0 0 0
- added joint r_foot_toe_joint: type fixed, parent Ankle_R_Roll_Link, child r_foot_toe, origin xyz=0.15484 0 -0.0725 rpy=0 0 0
- joint dummy_to_base_link: origin xyz=0 0.133 0.03605 rpy=0 0 0 -> xyz=-0.3605 0 -0.133 rpy=0 0 0

Commit message: 能走版本，walk缺插件未验证

File: src/humanoid_control/humanoid_legged_description/urdf/humanoid_legged_control_.urdf (robot description, URDF)
Before this commit: robot humanoid_legged_description, 18 links, 17 joints
Joints:
- joint dummy_to_base_link: origin xyz=-0.3605 0 -0.133 rpy=0 0 0 -> xyz=-0.3605 0 0.129 rpy=0 0 0
