Commit message: 冻结能走版本状态（含 ROS2 Jazzy / mujoco 3.14 迁移补丁）
工作区原有改动一并入库作为可复现基线：SafetyChecker/humanoidController
接口调整、task.info/task_.info 配置、humanoid_sim 暂停机制与接触缓存、
MJCF/URDF 脚底接触点、FootRollConstraint 改名、删除已废弃的
humanoid_controllers/config/controllers.yaml。

迁移补丁（Ubuntu 24.04 + ROS2 Jazzy + mujoco 3.14）：
- humanoid_controllers 显式 find_package/链接 pluginlib（Jazzy include
  布局变更后原传递包含断链，编译报 class_list_macros.hpp 缺失）
- install 规则去掉已删除的 config 目录（安装阶段报错）
- mujoco_base.py 相机调用改新签名 mjv_moveCamera(m, action, dx, dy, cam)
  —— 旧 5 参数调用在 mujoco>=3.2 抛 TypeError 并杀死仿真主循环
- 补 jrl-cmakemodules 的 cmake/coverage.cmake（vendored 拷贝缺失导致
  pinocchio 配置失败；被 pinocchio 自带 .gitignore 的 coverage* 规则
  隐藏，故 add -f 强制入库）

运行要点：仿真默认暂停（pause_flag=True），须在 MuJoCo 窗口按 SPACE
解除；/hwswitch 默认 false，须发布 true 才输出力矩指令。

验证：load_cheat_controller.launch.py 闭环成功行走（cheat 模式 +
trot），60s 全话题 rosbag 存于 experiments/walk_smoke_001/（不入库）。

Co-Authored-By: Claude Code <noreply@anthropic.com>

File: src/humanoid_control/humanoid_legged_description/urdf/humanoid_legged_control_.urdf (robot description, URDF)
Before this commit: robot humanoid_legged_description, 18 links, 17 joints
Joints:
- joint dummy_to_base_link: origin xyz=-0.3605 0 0.129 rpy=0 0 0 -> xyz=0.3605 0 0.129 rpy=0 0 0
