Commit message: C6 实机数据落地：real/ 42 run 分析 + 图表实机侧重绘
- real/（2026-10-22 批 42 run，基准 9 + 扰动 33）：README 说明口径与来源复核，
  rosbag 不入库（.gitignore）；run 级 analysis/ 由脚本可复算
- 分析链：analyze_real.py（42/42 VALID）→ make_real_stats.py → real_summary_stats.md
- 来源复核：real_provenance_review_2026-10-22.md §5（第四批 E1–E5/E7 全过、
  N3 谱系解除；残留 N1 SOC 不入文、E6 倒地同构如实写入）
- make_fig6.py 重写：仿真侧 sim_data/ + 实机侧 load_real()（mcap 直读，
  稳态窗复用 analyze_real.steady_window），fig6_1/2/3/4/5/6 全部 sim+real 重绘
- summary_stats.md/make_stats.py：路径迁移 sim_data/ 后的重算
- URDF effort 200→320（膝/髋俯仰）与 task_.info torqueLimitsTask 对齐（数据采集基线）
- 项目记忆：A3 状态、real/ 批次、画图脚本改造入档

Co-Authored-By: Claude Code <noreply@anthropic.com>

File: src/humanoid_control/humanoid_legged_description/urdf/humanoid_legged_origin.urdf (robot description, URDF)
Before this commit: robot humanoid_legged_description, 18 links, 17 joints
Joints:
- joint Hip_L_Pitch_Joint: limit lower=-0.78 upper=0.78 effort=200 velocity=5 -> lower=-0.78 upper=0.78 effort=320 velocity=5
- joint Hip_R_Pitch_Joint: limit lower=-0.78 upper=0.78 effort=200 velocity=5 -> lower=-0.78 upper=0.78 effort=320 velocity=5
- joint Knee_L_Pitch_Joint: limit lower=0 upper=1.2 effort=200 velocity=5 -> lower=0 upper=1.2 effort=320 velocity=5
- joint Knee_R_Pitch_Joint: limit lower=0 upper=1.2 effort=200 velocity=5 -> lower=0 upper=1.2 effort=320 velocity=5
